File: Proekt/Proekt.kicad_sch (KiCad schematic)
At the start: 36 parts, among them J1 RGB, J2 LX, J3 I2C, J4 UART, J5 USB_C_USB2.0, Q1 TEPT5700, SW1 RST, SW2 BTN, U1 ESP32-C3, U2 R1170H331B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

Commit message: dodadeno pcb design
Parts:
- R3: value 10k -> 100k
Connections:
- net +3V3 is gone; now on net +3.3V: C6.1, C7.1, J3.3 (Pin_3), J4.3 (Pin_3), R12.2, R13.2, U2.5 (VO), U3.5 (VBUS)
Other:
- note added: "Ambient light sensor"
- note added: "I2C header"
- note added: "Light sensor header"
- note added: "RGB LED"
- note added: "RGB LED header"
- note added: "UART header"
