File: Proekt/ProektBACKUP.kicad_pcb (KiCad board)
At the start: 2 copper layers, 40 x 40 mm, 36 parts, among them J1 RGB, J2 LX, J3 I2C, J4 UART, J5 USB_C_USB2.0, Q1 TEPT5700, SW1 RST, SW2 BTN, U1 ESP32-C3, U2 R1170H331B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

Commit message: dodadeno kabli
Routing:
- net GND: track 182.2 -> 175.8 mm
- net +3.3V: track 117.8 -> 115.8 mm
- net +5V: track 38.4 -> 36.8 mm
